Commit message: Balance_bot Version 2.0

File: robot/urdf/balancebot.urdf (robot description, URDF)
Before this commit: robot balancebot, 3 links, 2 joints
Links:
- link base_link: mass 100 -> 0.583032

File: urdf_test/urdf/balancebot.urdf (robot description, URDF)
Before this commit: robot balancebot, 3 links, 2 joints
Links:
- link base_link: mass 1.083032 -> 0.283032
